Commit message: add torque sensor to gazebo files

File: impedance_control/urdf/gazebo.urdf.xacro (robot description, xacro)
@@ -7,5 +7,5 @@
             <parameters>$(find impedance_control)/config/controllers.yaml</parameters>
         </plugin>
-        <!-- <plugin name="gazebo_ros2_force_torque" filename="libignition_ros2_sensors.so">
+        <!-- <plugin name="gazebo_ros2_force_torque" filename="libgazebo_ros2_sensors.so">
             <ros>
                 <namespace>/force_torque</namespace>
@@ -18,8 +18,4 @@
         <mu1>30.0</mu1>
         <mu2>30.0</mu2>
-        <material>Gazebo/Red</material>
-    </gazebo>
-    <gazebo reference="link1">
-        <material>Gazebo/Gray</material>
     </gazebo>
     <gazebo reference="link2">
@@ -28,8 +24,4 @@
         <mu1>30.0</mu1>
         <mu2>30.0</mu2>
-        <material>Gazebo/Red</material>
-    </gazebo>
-    <gazebo reference="link2">
-        <material>Gazebo/Gray</material>
     </gazebo>
     <gazebo reference="link3">
@@ -38,8 +30,4 @@
         <mu1>30.0</mu1>
         <mu2>30.0</mu2>
-        <material>Gazebo/Red</material>
-    </gazebo>
-    <gazebo reference="link3">
-        <material>Gazebo/Gray</material>
     </gazebo>
     <gazebo reference="joint1">

File: impedance_control/urdf/ros2_control.urdf.xacro (robot description, xacro)
@@ -14,4 +14,5 @@
                 </command_interface>
                 <command_interface name="velocity"/>
+                <command_interface name="effort"/>
                 <state_interface name="position">
                   <param name="initial_value">0.0</param>
@@ -27,4 +28,5 @@
                 </command_interface>
                 <command_interface name="velocity"/>
+                <command_interface name="effort"/>
                 <state_interface name="position">
                   <param name="initial_value">0.0</param>
@@ -40,4 +42,5 @@
                 </command_interface>
                 <command_interface name="velocity"/>
+                <command_interface name="effort"/>
                 <state_interface name="position">
                   <param name="initial_value">0.0</param>
