Commit message: add impedance and admittance code

File: impedance_control/urdf/3dof_manipulator.xacro (robot description, xacro)
@@ -5,5 +5,5 @@
   <!-- World -->
   <link name="world"/>
-  <!-- World fixed joint-->
+  <!-- World fixed joint -->
   <joint name="world_fixed" type="fixed">
     <origin xyz="0 0 0" rpy="0 0 0"/>
@@ -40,14 +40,13 @@
     <origin xyz="0 0 0.2" rpy="0 0 0"/>
     <axis xyz="0 0 1"/>
-    <limit lower="-1.57" upper="1.57" effort="10.0" velocity="1.0"/>
+    <limit lower="-3.14" upper="3.14" effort="10.0" velocity="1.0"/>
   </joint>
   <!-- Link 1 -->
   <link name="link1">
     <visual>
-      <origin xyz="0 0 0.1" rpy="0 0 0"/>
+      <origin xyz="0 0 0.25" rpy="0 0 0"/>
       <geometry>
         <cylinder radius="0.05" length="0.5"/>
       </geometry>
-      <origin xyz="0 0 0.25" rpy="0 0 0"/>
       <material name="green">
         <color rgba="0.0 1.0 0.0 1.0"/>
@@ -55,5 +54,5 @@
     </visual>
     <collision>
-      <origin xyz="0 0 0.1" rpy="0 0 0"/>
+      <origin xyz="0 0 0.25" rpy="0 0 0"/>
       <geometry>
         <cylinder radius="0.05" length="0.5"/>
@@ -61,5 +60,5 @@
     </collision>
     <inertial>
-      <mass value="0.5"/>
+      <mass value="1.0"/>
       <origin xyz="0 0 0.25" rpy="0 0 0"/>
       <inertia ixx="0.001" ixy="0.0" ixz="0.0" iyy="0.001" iyz="0.0" izz="0.001"/>
@@ -72,14 +71,13 @@
     <origin xyz="0 0 0.5" rpy="0 0 0"/>
     <axis xyz="0 1 0"/>
-    <limit lower="-1.57" upper="1.57" effort="10.0" velocity="1.0"/>
+    <limit lower="-3.14" upper="3.14" effort="10.0" velocity="1.0"/>
   </joint>
   <!-- Link 2 -->
   <link name="link2">
     <visual>
-      <origin xyz="0 0 0.1" rpy="0 0 0"/>
+      <origin xyz="0 0 0.25" rpy="0 0 0"/>
       <geometry>
         <cylinder radius="0.05" length="0.5"/>
       </geometry>
-      <origin xyz="0 0 0.25" rpy="0 0 0"/>
       <material name="red">
         <color rgba="1.0 0.0 0.0 1.0"/>
@@ -87,5 +85,5 @@
     </visual>
     <collision>
-      <origin xyz="0 0 0.1" rpy="0 0 0"/>
+      <origin xyz="0 0 0.25" rpy="0 0 0"/>
       <geometry>
         <cylinder radius="0.05" length="0.5"/>
@@ -93,5 +91,5 @@
     </collision>
     <inertial>
-      <mass value="0.5"/>
+      <mass value="1.0"/>
       <origin xyz="0 0 0.25" rpy="0 0 0"/>
       <inertia ixx="0.001" ixy="0.0" ixz="0.0" iyy="0.001" iyz="0.0" izz="0.001"/>
@@ -102,16 +100,15 @@
     <parent link="link2"/>
     <child link="link3"/>
-    <origin xyz="0 0 0.6" rpy="0 0 0"/>
+    <origin xyz="0 0 0.5" rpy="0 0 0"/>
     <axis xyz="1 0 0"/>
-    <limit lower="-1.57" upper="1.57" effort="10.0" velocity="1.0"/>
+    <limit lower="-3.14" upper="3.14" effort="10.0" velocity="1.0"/>
   </joint>
   <!-- Link 3 -->
   <link name="link3">
     <visual>
-      <origin xyz="0 0 0.1" rpy="0 0 0"/>
+      <origin xyz="0 0 0.25" rpy="0 0 0"/>
       <geometry>
         <cylinder radius="0.05" length="0.5"/>
       </geometry>
-      <origin xyz="0 0 0.25" rpy="0 0 0"/>
       <material name="yellow">
         <color rgba="1.0 1.0 0.0 1.0"/>
@@ -119,5 +116,5 @@
     </visual>
     <collision>
-      <origin xyz="0 0 0.1" rpy="0 0 0"/>
+      <origin xyz="0 0 0.25" rpy="0 0 0"/>
       <geometry>
         <cylinder radius="0.05" length="0.5"/>
@@ -125,5 +122,5 @@
     </collision>
     <inertial>
-      <mass value="0.5"/>
+      <mass value="1.0"/>
       <origin xyz="0 0 0.25" rpy="0 0 0"/>
       <inertia ixx="0.001" ixy="0.0" ixz="0.0" iyy="0.001" iyz="0.0" izz="0.001"/>
